File: hardware/clockInterface.sch (KiCad schematic (older format))
At the start: 9 parts, among them P501 CLOCK, SW501 SWITCH_INV, SW502 SWITCH_INV, SW503 SWITCH_INV, SW504 SWITCH_INV

Commit message: Added Reichelt/Mouser part numbers for all parts except ESP12-E/F
Parts:
- D501, D502: Reichelt (none) -> LED 3MM RT
- P501: Reichelt (none) -> AKL182-02 + AKL169-02
- R501, R502: Mouser (none) -> 603-RC0805JR-07220RL
- SW501, SW502, SW503, SW504: Mouser (none) -> 611-OS102011MS2QN1
Changed lines of the file:
@@
 F 2 "Capacitors_SMD:C_0805_HandSoldering" V 4380 2700 30  0001 C CNN
 F 3 "" H 4450 2700 30  0000 C CNN
+F 4 "603-RC0805JR-07220RL" V 4450 2700 60  0001 C CNN "Mouser"
 	1    4450 2700
 	0    1    1    0
@@
 F 2 "Capacitors_SMD:C_0805_HandSoldering" V 4380 3500 30  0001 C CNN
 F 3 "" H 4450 3500 30  0000 C CNN
+F 4 "603-RC0805JR-07220RL" V 4450 3500 60  0001 C CNN "Mouser"
 	1    4450 3500
 	0    1    1    0
@@
 F 2 "myFootprints:LED_D3.0mm" H 5000 3100 60  0001 C CNN
 F 3 "" H 5000 3100 60  0000 C CNN
+F 4 "LED 3MM RT" H 5000 3100 60  0001 C CNN "Reichelt"
 	1    5000 3100
 	0    1    1    0
@@
 F 2 "myFootprints:LED_D3.0mm" H 5300 3100 60  0001 C CNN
 F 3 "" H 5300 3100 60  0000 C CNN
+F 4 "LED 3MM RT" H 5300 3100 60  0001 C CNN "Reichelt"
 	1    5300 3100
 	0    -1   -1   0
@@
 F 2 "myFootprints:AKL183-02" H 6150 3100 60  0001 C CNN
 F 3 "" H 6150 3100 60  0001 C CNN
+F 4 "AKL182-02 + AKL169-02" V 6150 3100 60  0001 C CNN "Reichelt"
 	1    6150 3100
 	1    0    0    -1
@@
 F 2 "myFootprints:OS102011MS2Q" H 4500 4100 60  0001 C CNN
 F 3 "" H 4500 4100 60  0000 C CNN
+F 4 "611-OS102011MS2QN1" H 4500 4100 60  0001 C CNN "Mouser"
 	1    4500 4100
 	1    0    0    -1
@@
 F 2 "myFootprints:OS102011MS2Q" H 4500 4600 60  0001 C CNN
 F 3 "" H 4500 4600 60  0000 C CNN
+F 4 "611-OS102011MS2QN1" H 4500 4600 60  0001 C CNN "Mouser"
 	1    4500 4600
 	1    0    0    -1
@@
 F 2 "myFootprints:OS102011MS2Q" H 4500 5100 60  0001 C CNN
 F 3 "" H 4500 5100 60  0000 C CNN
+F 4 "611-OS102011MS2QN1" H 4500 5100 60  0001 C CNN "Mouser"
 	1    4500 5100
 	1    0    0    -1
@@
 F 2 "myFootprints:OS102011MS2Q" H 4500 5600 60  0001 C CNN
 F 3 "" H 4500 5600 60  0000 C CNN
+F 4 "611-OS102011MS2QN1" H 4500 5600 60  0001 C CNN "Mouser"
 	1    4500 5600
 	1    0    0    -1
