File: hardware/loconet-interface.sch (KiCad schematic (older format))
At the start: 24 parts, among them J301 Molex 95501-6669, K301 TERMINATION, Q301 BC817-40, Q302 BC817-40, Q303 BC817-40, U301 TC1240

Commit message: Added Reichelt/Mouser part numbers for all parts except ESP12-E/F
Parts:
- C301: Reichelt (none) -> NPO-G0805 1,0N
- C302: Reichelt (none) -> NPO-G0805 47P
- C303: Reichelt (none) -> X7R-G0805 100N
- C304, C305: Reichelt (none) -> X5R-G0805 22/25
- J301: Farnell 2060710 -> (none); Mouser (none) -> 538-95501-6669
- K301: Reichelt (none) -> RND 205-00631
- R301: Mouser (none) -> 603-RC0805JR-074K7L
- R302, R304, R310: Mouser (none) -> 603-RC0805JR-0747KL
- R303: Mouser (none) -> 603-RC0805JR-0747RL
- R305: Mouser (none) -> 603-RC0805JR-072K2L
- R306: Mouser (none) -> 603-RC0805JR-0782KL
- R307, R308: Mouser (none) -> 603-RC0805JR-0712RL
- R309: Mouser (none) -> 603-RC0805JR-07100KL
- U301: Mouser (none) -> 579-TC1240ECHTR
Changed lines of the file:
@@
 F 2 "myFootprints:Molex_95501-6669" H 7350 2600 60  0001 C CNN
 F 3 "" H 7350 2600 60  0001 C CNN
-F 4 "2060710" H 7350 2600 60  0001 C CNN "Farnell"
+F 4 "538-95501-6669" H 7350 2600 60  0001 C CNN "Mouser"
 	1    7350 2600
 	0    1    1    0
@@
 F 2 "Capacitors_SMD:C_0805_HandSoldering" V 5830 4150 30  0001 C CNN
 F 3 "" H 5900 4150 30  0000 C CNN
+F 4 "603-RC0805JR-0712RL" V 5900 4150 60  0001 C CNN "Mouser"
 	1    5900 4150
 	1    0    0    -1
@@
 F 2 "Capacitors_SMD:C_0805_HandSoldering" V 5830 4850 30  0001 C CNN
 F 3 "" H 5900 4850 30  0000 C CNN
+F 4 "603-RC0805JR-0712RL" V 5900 4850 60  0001 C CNN "Mouser"
 	1    5900 4850
 	1    0    0    -1
@@
 F 2 "Capacitors_SMD:C_0805_HandSoldering" H 6238 4650 30  0001 C CNN
 F 3 "" H 6200 4800 60  0000 C CNN
+F 4 "NPO-G0805 47P" H 6200 4800 60  0001 C CNN "Reichelt"
 	1    6200 4800
 	1    0    0    -1
@@
 F 2 "Capacitors_SMD:C_0805_HandSoldering" V 5480 5200 30  0001 C CNN
 F 3 "" H 5550 5200 30  0000 C CNN
+F 4 "603-RC0805JR-0782KL" V 5550 5200 60  0001 C CNN "Mouser"
 	1    5550 5200
 	0    1    1    0
@@
 F 2 "Capacitors_SMD:C_0805_HandSoldering" V 4780 5200 30  0001 C CNN
 F 3 "" H 4850 5200 30  0000 C CNN
+F 4 "603-RC0805JR-0747KL" V 4850 5200 60  0001 C CNN "Mouser"
 	1    4850 5200
 	0    1    1    0
@@
 F 2 "Capacitors_SMD:C_0805_HandSoldering" V 5080 5700 30  0001 C CNN
 F 3 "" H 5150 5700 30  0000 C CNN
+F 4 "603-RC0805JR-072K2L" V 5150 5700 60  0001 C CNN "Mouser"
 	1    5150 5700
 	0    1    1    0
@@
 F 2 "Capacitors_SMD:C_0805_HandSoldering" V 4130 5550 30  0001 C CNN
 F 3 "" H 4200 5550 30  0000 C CNN
+F 4 "603-RC0805JR-0747KL" V 4200 5550 60  0001 C CNN "Mouser"
 	1    4200 5550
 	-1   0    0    1
@@
 F 2 "Capacitors_SMD:C_0805_HandSoldering" V 7580 5650 30  0001 C CNN
 F 3 "" H 7650 5650 30  0000 C CNN
+F 4 "603-RC0805JR-0747KL" V 7650 5650 60  0001 C CNN "Mouser"
 	1    7650 5650
 	1    0    0    -1
@@
 F 2 "Capacitors_SMD:C_0805_HandSoldering" V 7580 4850 30  0001 C CNN
 F 3 "" H 7650 4850 30  0000 C CNN
+F 4 "603-RC0805JR-07100KL" V 7650 4850 60  0001 C CNN "Mouser"
 	1    7650 4850
 	1    0    0    -1
@@
 F 2 "Capacitors_SMD:C_0805_HandSoldering" H 7988 5500 30  0001 C CNN
 F 3 "" H 7950 5650 60  0000 C CNN
+F 4 "X7R-G0805 100N" H 7950 5650 60  0001 C CNN "Reichelt"
 	1    7950 5650
 	1    0    0    -1
@@
 F 2 "Capacitors_SMD:C_0805_HandSoldering" H 5188 5850 30  0001 C CNN
 F 3 "" H 5150 6000 60  0000 C CNN
+F 4 "NPO-G0805 1,0N" H 5150 6000 60  0001 C CNN "Reichelt"
 	1    5150 6000
 	0    1    1    0
@@
 F 2 "Capacitors_SMD:C_0805_HandSoldering" V 4130 1850 30  0001 C CNN
 F 3 "" H 4200 1850 30  0000 C CNN
+F 4 "603-RC0805JR-074K7L" V 4200 1850 60  0001 C CNN "Mouser"
 	1    4200 1850
 	-1   0    0    1
@@
 F 2 "Capacitors_SMD:C_0805_HandSoldering" V 4630 2950 30  0001 C CNN
 F 3 "" H 4700 2950 30  0000 C CNN
+F 4 "603-RC0805JR-0747RL" V 4700 2950 60  0001 C CNN "Mouser"
 	1    4700 2950
 	-1   0    0    1
@@
 F 2 "Pin_Headers:Pin_Header_Straight_1x03_Pitch2.54mm" H 3750 1300 60  0001 C CNN
 F 3 "" H 3750 1300 60  0001 C CNN
+F 4 "RND 205-00631" V 3750 1300 60  0001 C CNN "Reichelt"
 	1    3750 1300
 	-1   0    0    1
@@
 F 2 "TO_SOT_Packages_SMD:SOT-23-6_Handsoldering" H 2300 2400 60  0001 C CNN
 F 3 "" H 2300 2400 60  0001 C CNN
+F 4 "579-TC1240ECHTR" H 2300 2400 60  0001 C CNN "Mouser"
 	1    2300 2400
 	1    0    0    -1
@@
 F 2 "Capacitors_SMD:C_0805_HandSoldering" H 1338 2400 30  0001 C CNN
 F 3 "" H 1300 2550 60  0000 C CNN
+F 4 "X5R-G0805 22/25" H 1300 2550 60  0001 C CNN "Reichelt"
 	1    1300 2550
 	1    0    0    -1
@@
 F 2 "Capacitors_SMD:C_0805_HandSoldering" H 3238 2250 30  0001 C CNN
 F 3 "" H 3200 2400 60  0000 C CNN
+F 4 "X5R-G0805 22/25" H 3200 2400 60  0001 C CNN "Reichelt"
 	1    3200 2400
 	1    0    0    -1
