File: hardware/wfred_loconet_clock.sch (KiCad schematic (older format))
At the start: 8 parts, among them U101 L6920D

Commit message: Added Reichelt/Mouser part numbers for all parts except ESP12-E/F
Parts:
- B101: Reichelt (none) -> KEYSTONE 1013
- L101: Reichelt L-PISM 22µ -> L-242418FPS 22µ
- U101: Mouser (none) -> 511-L6920DTR
Changed lines of the file:
@@
 F 2 "myFootprints:L_2424_HandSoldering" H 4300 1400 60  0001 C CNN
 F 3 "" H 4300 1400 60  0000 C CNN
-F 4 "L-PISM 22µ" V 4300 1400 60  0001 C CNN "Reichelt"
+F 4 "L-242418FPS 22µ" V 4300 1400 60  0001 C CNN "Reichelt"
 	1    4300 1400
 	1    0    0    -1
@@
 F 3 "" H 4300 2500 60  0001 C CNN
 F 4 "L 6920 D" H 4300 2500 60  0001 C CNN "Reichelt"
+F 5 "511-L6920DTR" H 4300 2500 60  0001 C CNN "Mouser"
 	1    4300 2500
 	1    0    0    -1
@@
 F 2 "myFootprints:KEYSTONE1013" H 1200 4900 60  0001 C CNN
 F 3 "" H 1200 4900 60  0001 C CNN
+F 4 "KEYSTONE 1013" H 1200 4900 60  0001 C CNN "Reichelt"
 	1    1200 4900
 	0    1    1    0
