File: hardware/wfred-controller_rev2.sch (KiCad schematic (older format))
At the start: 13 parts, among them IC201 ATMEGA328P-A, P201 ISP, X201 14.7456MHz

Commit message: Fixed PCB: Added proper GND connection...
...and removed unrequired power measurement resistors
Parts:
- removed R202, R203: 100k, Capacitors_SMD:C_0805_HandSoldering, symbol R
Connections:
- wire segments 73 -> 70
- no-connect marks 0 -> 1
Changed lines of the file:
@@
-$EndComp
-$Comp
-L R R202
-U 1 1 5BE0AFE0
-P 2800 4050
-F 0 "R202" V 2880 4050 40  0000 C CNN
-F 1 "100k" V 2807 4051 40  0000 C CNN
-F 2 "Capacitors_SMD:C_0805_HandSoldering" V 2730 4050 30  0001 C CNN
-F 3 "" H 2800 4050 30  0000 C CNN
-	1    2800 4050
-	-1   0    0    -1
-$EndComp
-$Comp
-L R R203
-U 1 1 5BE0B09F
-P 2800 5050
-F 0 "R203" V 2880 5050 40  0000 C CNN
-F 1 "100k" V 2807 5051 40  0000 C CNN
-F 2 "Capacitors_SMD:C_0805_HandSoldering" V 2730 5050 30  0001 C CNN
-F 3 "" H 2800 5050 30  0000 C CNN
-	1    2800 5050
-	-1   0    0    -1
 $EndComp
 $Comp
 L +BATT #PWR033
 U 1 1 5BE0B208
-P 2800 3100
-F 0 "#PWR033" H 2800 3050 20  0001 C CNN
-F 1 "+BATT" H 2800 3200 30  0000 C CNN
-F 2 "" H 2800 3100 60  0001 C CNN
-F 3 "" H 2800 3100 60  0001 C CNN
-	1    2800 3100
+P 3300 3100
+F 0 "#PWR033" H 3300 3050 20  0001 C CNN
+F 1 "+BATT" H 3300 3200 30  0000 C CNN
+F 2 "" H 3300 3100 60  0001 C CNN
+F 3 "" H 3300 3100 60  0001 C CNN
+	1    3300 3100
 	-1   0    0    -1
 $EndComp
@@
 Wire Wire Line
 	5900 5100 6600 5100
-Wire Wire Line
-	2800 4300 2800 4800
 Wire Wire Line
 	5900 4550 6600 4550
@@
 	5000 2400 5900 2400
 Wire Wire Line
-	2800 4550 4000 4550
-Wire Wire Line
-	2800 3100 2800 3800
-Wire Wire Line
-	2800 3200 4000 3200
-Connection ~ 2800 3200
-Wire Wire Line
 	4000 3300 3850 3300
 Wire Wire Line
@@
 	3850 3500 4000 3500
 Connection ~ 3850 3300
-$Comp
-L GND-RESCUE-wfred_rev2 #PWR034
-U 1 1 5BE232F3
-P 2800 5700
-F 0 "#PWR034" H 2800 5700 30  0001 C CNN
-F 1 "GND" H 2800 5630 30  0001 C CNN
-F 2 "" H 2800 5700 60  0001 C CNN
-F 3 "" H 2800 5700 60  0001 C CNN
-	1    2800 5700
-	1    0    0    -1
-$EndComp
-Wire Wire Line
-	2800 5300 2800 5700
 Wire Wire Line
 	3300 5500 4000 5500
@@
 Wire Wire Line
 	3800 4650 4000 4650
-Connection ~ 2800 4550
+NoConn ~ 4000 4550
+Wire Wire Line
+	4000 3200 3300 3200
+Wire Wire Line
+	3300 3200 3300 3100
 $EndSCHEMATC

Commit message: Change TX series resistor value to 220R...
...as per the working prototype
Parts:
- R204: value 10k -> 220R
Changed lines of the file:
@@
 P 7450 4900
 F 0 "R204" V 7530 4900 40  0000 C CNN
-F 1 "10k" V 7457 4901 40  0000 C CNN
+F 1 "220R" V 7457 4901 40  0000 C CNN
 F 2 "Capacitors_SMD:C_0805_HandSoldering" V 7380 4900 30  0001 C CNN
 F 3 "" H 7450 4900 30  0000 C CNN

Commit message: Rename labels, cleanup schematics
Connections:
- net labels added: F0_F2_F5_F8, F1_F4_F7_ESTOP, F3_F6_SHIFT
- net labels removed: F0_SHIFT_ESTOP, F1_F2_F3_F4, F5_F6_F7_F8
Changed lines of the file:
@@
 L C-RESCUE-wfred_rev2 C205
 U 1 1 5920CFB6
-P 10200 3100
+P 8900 3100
 AR Path="/5920CFB6" Ref="C205"  Part="1"
 AR Path="/5920C945/5920CFB6" Ref="C205"  Part="1"
-F 0 "C205" H 10200 3200 40  0000 L CNN
-F 1 "22p" H 10206 3015 40  0000 L CNN
-F 2 "Capacitors_SMD:C_0805_HandSoldering" H 10238 2950 30  0001 C CNN
-F 3 "" H 10200 3100 60  0000 C CNN
-F 4 "NPO-G0805 22P" H 10200 3100 60  0001 C CNN "Reichelt"
-	1    10200 3100
+F 0 "C205" H 8900 3200 40  0000 L CNN
+F 1 "22p" H 8906 3015 40  0000 L CNN
+F 2 "Capacitors_SMD:C_0805_HandSoldering" H 8938 2950 30  0001 C CNN
+F 3 "" H 8900 3100 60  0000 C CNN
+F 4 "NPO-G0805 22P" H 8900 3100 60  0001 C CNN "Reichelt"
+	1    8900 3100
 	0    -1   1    0
 $EndComp
@@
 L C-RESCUE-wfred_rev2 C206
 U 1 1 5920D023
-P 10200 3900
+P 8900 3900
 AR Path="/5920D023" Ref="C206"  Part="1"
 AR Path="/5920C945/5920D023" Ref="C206"  Part="1"
-F 0 "C206" H 10200 4000 40  0000 L CNN
-F 1 "22p" H 10206 3815 40  0000 L CNN
-F 2 "Capacitors_SMD:C_0805_HandSoldering" H 10238 3750 30  0001 C CNN
-F 3 "" H 10200 3900 60  0000 C CNN
-F 4 "NPO-G0805 22P" H 10200 3900 60  0001 C CNN "Reichelt"
-	1    10200 3900
+F 0 "C206" H 8900 4000 40  0000 L CNN
+F 1 "22p" H 8906 3815 40  0000 L CNN
+F 2 "Capacitors_SMD:C_0805_HandSoldering" H 8938 3750 30  0001 C CNN
+F 3 "" H 8900 3900 60  0000 C CNN
+F 4 "NPO-G0805 22P" H 8900 3900 60  0001 C CNN "Reichelt"
+	1    8900 3900
 	0    -1   1    0
 $EndComp
@@
 L GND-RESCUE-wfred_rev2 #PWR027
 U 1 1 5920D54C
-P 10600 4100
-F 0 "#PWR027" H 10600 4100 30  0001 C CNN
-F 1 "GND" H 10600 4030 30  0001 C CNN
-F 2 "" H 10600 4100 60  0001 C CNN
-F 3 "" H 10600 4100 60  0001 C CNN
-	1    10600 4100
+P 9300 4100
+F 0 "#PWR027" H 9300 4100 30  0001 C CNN
+F 1 "GND" H 9300 4030 30  0001 C CNN
+F 2 "" H 9300 4100 60  0001 C CNN
+F 3 "" H 9300 4100 60  0001 C CNN
+	1    9300 4100
 	-1   0    0    -1
 $EndComp
@@
 	1    0    0    -1
 $EndComp
-Text GLabel 7900 4900 2    60   Output ~ 0
+Text GLabel 8200 4900 2    60   Output ~ 0
 THIS_TXD
 Text GLabel 6600 4800 2    60   Input ~ 0
@@
 L myCRYSTAL X201
 U 1 1 5A171DD9
-P 9700 3500
-F 0 "X201" H 9700 3650 60  0000 C CNN
-F 1 "14.7456MHz" H 9700 3350 60  0000 C CNN
-F 2 "Crystals:Crystal_SMD_TXC_7M-4pin_3.2x2.5mm_HandSoldering" H 9700 3500 60  0001 C CNN
-F 3 "" H 9700 3500 60  0000 C CNN
-F 4 "449-LFXTAL036338CUTT" H 9700 3500 60  0001 C CNN "Mouser"
-	1    9700 3500
+P 8400 3500
+F 0 "X201" H 8400 3650 60  0000 C CNN
+F 1 "14.7456MHz" H 8400 3350 60  0000 C CNN
+F 2 "Crystals:Crystal_SMD_TXC_7M-4pin_3.2x2.5mm_HandSoldering" H 8400 3500 60  0001 C CNN
+F 3 "" H 8400 3500 60  0000 C CNN
+F 4 "449-LFXTAL036338CUTT" H 8400 3500 60  0001 C CNN "Mouser"
+	1    8400 3500
 	0    1    1    0
 $EndComp
@@
 L GND-RESCUE-wfred_rev2 #PWR030
 U 1 1 5A171EC6
-P 9500 4100
-F 0 "#PWR030" H 9500 4100 30  0001 C CNN
-F 1 "GND" H 9500 4030 30  0001 C CNN
-F 2 "" H 9500 4100 60  0001 C CNN
-F 3 "" H 9500 4100 60  0001 C CNN
-	1    9500 4100
+P 8200 4100
+F 0 "#PWR030" H 8200 4100 30  0001 C CNN
+F 1 "GND" H 8200 4030 30  0001 C CNN
+F 2 "" H 8200 4100 60  0001 C CNN
+F 3 "" H 8200 4100 60  0001 C CNN
+	1    8200 4100
 	-1   0    0    -1
 $EndComp
@@
 L GND-RESCUE-wfred_rev2 #PWR031
 U 1 1 5A171EEF
-P 9300 3300
-F 0 "#PWR031" H 9300 3300 30  0001 C CNN
-F 1 "GND" H 9300 3230 30  0001 C CNN
-F 2 "" H 9300 3300 60  0001 C CNN
-F 3 "" H 9300 3300 60  0001 C CNN
-	1    9300 3300
+P 8000 3300
+F 0 "#PWR031" H 8000 3300 30  0001 C CNN
+F 1 "GND" H 8000 3230 30  0001 C CNN
+F 2 "" H 8000 3300 60  0001 C CNN
+F 3 "" H 8000 3300 60  0001 C CNN
+	1    8000 3300
 	-1   0    0    -1
 $EndComp
@@
 $EndComp
 Wire Wire Line
-	9700 3100 9700 3200
-Wire Wire Line
-	9700 3800 9700 3900
-Wire Wire Line
-	5900 3900 10000 3900
+	8400 3100 8400 3200
+Wire Wire Line
+	8400 3800 8400 3900
+Wire Wire Line
+	5900 3900 8700 3900
 Wire Wire Line
 	5600 1600 5600 1800
@@
 Connection ~ 5300 2400
 Connection ~ 5600 2400
-Connection ~ 9700 3100
-Connection ~ 9700 3900
-Wire Wire Line
-	10400 3100 10600 3100
-Wire Wire Line
-	10600 3100 10600 4100
-Wire Wire Line
-	10400 3900 10600 3900
-Connection ~ 10600 3900
+Connection ~ 8400 3100
+Connection ~ 8400 3900
+Wire Wire Line
+	9100 3100 9300 3100
+Wire Wire Line
+	9300 3100 9300 4100
+Wire Wire Line
+	9100 3900 9300 3900
+Connection ~ 9300 3900
 Wire Wire Line
 	3300 3700 3300 4000
@@
 Connection ~ 3900 2200
 Wire Wire Line
-	9500 3200 9500 3000
-Wire Wire Line
-	9500 3000 9300 3000
-Wire Wire Line
-	9300 3000 9300 3300
-Wire Wire Line
-	9500 3800 9500 4100
-Wire Wire Line
-	9100 3100 9100 3800
-Wire Wire Line
-	9100 3100 10000 3100
+	8200 3200 8200 3000
+Wire Wire Line
+	8200 3000 8000 3000
+Wire Wire Line
+	8000 3000 8000 3300
+Wire Wire Line
+	8200 3800 8200 4100
+Wire Wire Line
+	7800 3100 7800 3800
+Wire Wire Line
+	7800 3100 8700 3100
 Wire Wire Line
 	5900 4350 6600 4350
@@
 	5900 4550 6600 4550
 Wire Wire Line
-	7700 4900 7900 4900
+	7700 4900 8200 4900
 $Comp
 L ATMEGA328P-A IC201
@@
 	5900 4650 6600 4650
 Wire Wire Line
-	9100 3800 5900 3800
+	7800 3800 5900 3800
 Text GLabel 6600 4450 2    60   Output ~ 0
 LED_STOP
@@
 DIRECTION
 Text GLabel 6600 3400 2    60   Output ~ 0
-F5_F6_F7_F8
+F3_F6_SHIFT
 Text GLabel 6600 3300 2    60   Output ~ 0
-F1_F2_F3_F4
+F0_F2_F5_F8
 Text GLabel 6600 3200 2    60   Output ~ 0
-F0_SHIFT_ESTOP
+F1_F4_F7_ESTOP
 Wire Wire Line
 	3800 4650 4000 4650
 NoConn ~ 4000 4550
 Wire Wire Line
-	4000 3200 3300 3200
+	3300 3200 4000 3200
 Wire Wire Line
 	3300 3200 3300 3100
