File: hardware/wfred-controller_rev2.sch (KiCad schematic (older format))
At the start: 12 parts, among them IC201 ATMEGA328P-A, P201 ISP, X201 14.7456MHz

Commit message: Fixed merge conflicts from last commit in pcbNew
Connections:
- wire segments 72 -> 74
Changed lines of the file:
@@
 	7800 4600 7800 4900
 Connection ~ 7800 4900
+Wire Wire Line
+	6300 3600 5900 3600
+Wire Wire Line
+	6400 3700 5900 3700
 $EndSCHEMATC

Commit message: Updated schematic and PCB for kicad 5.1.4
Parts:
- C201, C202, C203, C205, C206, C207: symbol C-RESCUE-wfred_rev2 -> wfred_rev2-rescue:C-RESCUE-wfred_rev2
- D201: symbol BAR43 -> my_devices:BAR43
- IC201: symbol ATMEGA328P-A -> atmel:ATMEGA328P-A
- P201: symbol CONN_3X2 -> conn:CONN_3X2
- R201: symbol R-RESCUE-wfred_rev2 -> wfred_rev2-rescue:R-RESCUE-wfred_rev2
- R204: symbol R -> device:R
- X201: symbol myCRYSTAL -> my_devices:myCRYSTAL
Connections:
- wire segments 74 -> 93
Changed lines of the file:
@@
-EESchema Schematic File Version 2
-LIBS:wfred_rev2-rescue
-LIBS:power
-LIBS:device
-LIBS:transistors
-LIBS:conn
-LIBS:linear
-LIBS:regul
-LIBS:74xx
-LIBS:cmos4000
-LIBS:adc-dac
-LIBS:memory
-LIBS:xilinx
-LIBS:microcontrollers
-LIBS:dsp
-LIBS:microchip
-LIBS:analog_switches
-LIBS:motorola
-LIBS:texas
-LIBS:intel
-LIBS:audio
-LIBS:interface
-LIBS:digital-audio
-LIBS:philips
-LIBS:display
-LIBS:cypress
-LIBS:siliconi
-LIBS:opto
-LIBS:atmel
-LIBS:contrib
-LIBS:valves
-LIBS:my_devices
-LIBS:ESP8266
-LIBS:LDL1117S30R
-LIBS:MCP73831T-2ACI_OT
-LIBS:NCV8161BSN300T1G
+EESchema Schematic File Version 4
 LIBS:wfred_rev2-cache
-EELAYER 25 0
+EELAYER 30 0
 EELAYER END
 $Descr A4 11693 8268
@@
 $EndDescr
 $Comp
-L C-RESCUE-wfred_rev2 C205
+L wfred_rev2-rescue:C-RESCUE-wfred_rev2 C205
 U 1 1 5920CFB6
 P 8900 3100
@@
 $EndComp
 $Comp
-L C-RESCUE-wfred_rev2 C206
+L wfred_rev2-rescue:C-RESCUE-wfred_rev2 C206
 U 1 1 5920D023
 P 8900 3900
@@
 $EndComp
 $Comp
-L C-RESCUE-wfred_rev2 C202
+L wfred_rev2-rescue:C-RESCUE-wfred_rev2 C202
 U 1 1 5920D0A7
 P 5300 2000
@@
 $EndComp
 $Comp
-L C-RESCUE-wfred_rev2 C203
+L wfred_rev2-rescue:C-RESCUE-wfred_rev2 C203
 U 1 1 5920E33B
 P 5600 2000
@@
 $EndComp
 $Comp
-L C-RESCUE-wfred_rev2 C201
+L wfred_rev2-rescue:C-RESCUE-wfred_rev2 C201
 U 1 1 5920E47C
 P 3300 4200
@@
 $EndComp
 $Comp
-L CONN_3X2 P201
+L conn:CONN_3X2 P201
 U 1 1 5920E592
 P 4400 2150
@@
 $EndComp
 $Comp
-L R-RESCUE-wfred_rev2 R201
+L wfred_rev2-rescue:R-RESCUE-wfred_rev2 R201
 U 1 1 5920FD60
 P 4450 1600
@@
 MOSI
 $Comp
-L PWR_FLAG #FLG026
+L power:PWR_FLAG #FLG026
 U 1 1 59214642
 P 3300 3700
@@
 $EndComp
 $Comp
-L GND-RESCUE-wfred_rev2 #PWR027
+L wfred_rev2-rescue:GND-RESCUE-wfred_rev2 #PWR027
 U 1 1 5920D54C
 P 9300 4100
@@
 $EndComp
 $Comp
-L GND-RESCUE-wfred_rev2 #PWR028
+L wfred_rev2-rescue:GND-RESCUE-wfred_rev2 #PWR028
 U 1 1 5920D60E
 P 5300 2600
@@
 SPEED
 $Comp
-L GND-RESCUE-wfred_rev2 #PWR029
+L wfred_rev2-rescue:GND-RESCUE-wfred_rev2 #PWR029
 U 1 1 592F4690
 P 3300 5700
@@
 F2
 $Comp
-L myCRYSTAL X201
+L my_devices:myCRYSTAL X201
 U 1 1 5A171DD9
 P 8400 3500
@@
 $EndComp
 $Comp
-L GND-RESCUE-wfred_rev2 #PWR030
+L wfred_rev2-rescue:GND-RESCUE-wfred_rev2 #PWR030
 U 1 1 5A171EC6
 P 8200 4100
@@
 $EndComp
 $Comp
-L GND-RESCUE-wfred_rev2 #PWR031
+L wfred_rev2-rescue:GND-RESCUE-wfred_rev2 #PWR031
 U 1 1 5A171EEF
 P 8000 3300
@@
 ESP_ENABLE
 $Comp
-L +BATT #PWR032
+L power:+BATT #PWR032
 U 1 1 5BE0AEFB
 P 5400 1400
@@
 $EndComp
 $Comp
-L +BATT #PWR033
+L power:+BATT #PWR033
 U 1 1 5BE0B208
 P 3300 3100
@@
 SPEED_POWER
 $Comp
-L R R204
+L device:R R204
 U 1 1 5BE0AFA5
 P 7450 4900
@@
 	8400 3800 8400 3900
 Wire Wire Line
-	5900 3900 8700 3900
+	5900 3900 8400 3900
 Wire Wire Line
 	5600 1600 5600 1800
@@
 Connection ~ 5600 1600
 Wire Wire Line
-	5300 2200 5300 2600
+	5300 2200 5300 2400
 Wire Wire Line
 	5600 2400 5600 2200
@@
 	9100 3100 9300 3100
 Wire Wire Line
-	9300 3100 9300 4100
+	9300 3100 9300 3900
 Wire Wire Line
 	9100 3900 9300 3900
 Connection ~ 9300 3900
 Wire Wire Line
-	3300 3700 3300 4000
-Wire Wire Line
-	3300 4400 3300 5700
+	3300 3700 3300 3800
+Wire Wire Line
+	3300 4400 3300 5500
 Wire Wire Line
 	5000 2000 4800 2000
@@
 	5900 4250 6600 4250
 Wire Wire Line
-	5900 3500 6600 3500
+	5900 3500 6200 3500
 Wire Wire Line
 	5000 2200 5000 2400
@@
 	7800 3100 7800 3800
 Wire Wire Line
-	7800 3100 8700 3100
+	7800 3100 8400 3100
 Wire Wire Line
 	5900 4350 6600 4350
@@
 	5900 3400 6600 3400
 Wire Wire Line
-	3800 2200 4000 2200
+	3800 2200 3900 2200
 Wire Wire Line
 	5900 5100 6600 5100
@@
 	5900 4550 6600 4550
 Wire Wire Line
-	7700 4900 8200 4900
-$Comp
-L ATMEGA328P-A IC201
+	7700 4900 7800 4900
+$Comp
+L atmel:ATMEGA328P-A IC201
 U 1 1 5BE1F936
 P 4900 4300
@@
 	5900 1600 5900 1800
 Wire Wire Line
-	4700 1600 5900 1600
-$Comp
-L C-RESCUE-wfred_rev2 C207
+	4700 1600 5000 1600
+$Comp
+L wfred_rev2-rescue:C-RESCUE-wfred_rev2 C207
 U 1 1 5BDF9383
 P 5900 2000
@@
 $EndComp
 Wire Wire Line
-	5000 2400 5900 2400
+	5000 2400 5300 2400
 Wire Wire Line
 	4000 3300 3850 3300
 Wire Wire Line
-	3850 3200 3850 3500
+	3850 3200 3850 3300
 Connection ~ 3850 3200
 Wire Wire Line
@@
 Connection ~ 3850 3300
 Wire Wire Line
-	3300 5500 4000 5500
+	3300 5500 3900 5500
 Connection ~ 3300 5500
 Wire Wire Line
 	4000 5400 3900 5400
 Wire Wire Line
-	3900 5300 3900 5500
+	3900 5300 3900 5400
 Connection ~ 3900 5500
 Wire Wire Line
@@
 NoConn ~ 4000 4550
 Wire Wire Line
-	3300 3200 4000 3200
+	3300 3200 3850 3200
 Wire Wire Line
 	3300 3200 3300 3100
 $Comp
-L BAR43 D201
+L my_devices:BAR43 D201
 U 1 1 5CD177D6
 P 8100 4600
@@
 $EndComp
 $Comp
-L VCC #PWR034
+L power:VCC #PWR034
 U 1 1 5CD17879
 P 8500 4400
@@
 Wire Wire Line
 	6400 3700 5900 3700
+Wire Wire Line
+	5600 1600 5900 1600
+Wire Wire Line
+	5300 2400 5300 2600
+Wire Wire Line
+	5300 2400 5600 2400
+Wire Wire Line
+	5600 2400 5900 2400
+Wire Wire Line
+	8400 3100 8700 3100
+Wire Wire Line
+	8400 3900 8700 3900
+Wire Wire Line
+	9300 3900 9300 4100
+Wire Wire Line
+	5000 1600 5300 1600
+Wire Wire Line
+	5300 1600 5400 1600
+Wire Wire Line
+	3300 3800 3300 4000
+Wire Wire Line
+	5400 1600 5600 1600
+Wire Wire Line
+	3900 2200 4000 2200
+Wire Wire Line
+	6200 3500 6600 3500
+Wire Wire Line
+	3850 3200 4000 3200
+Wire Wire Line
+	3850 3300 3850 3500
+Wire Wire Line
+	3300 5500 3300 5700
+Wire Wire Line
+	3900 5500 4000 5500
+Wire Wire Line
+	3900 5400 3900 5500
+Wire Wire Line
+	7800 4900 8200 4900
 $EndSCHEMATC

Commit message: Opened schematic and PCB in new kicad version
...causing a couple of changes to libraries and schematic and PCB files
Parts:
- IC201: symbol atmel:ATMEGA328P-A -> wfred_rev2-rescue:ATMEGA328P-A-atmel
- P201: symbol conn:CONN_3X2 -> wfred_rev2-rescue:CONN_3X2-conn
- R204: symbol device:R -> wfred_rev2-rescue:R-device
Changed lines of the file:
@@
 EESchema Schematic File Version 4
-LIBS:wfred_rev2-cache
 EELAYER 30 0
 EELAYER END
@@
 $EndComp
 $Comp
-L conn:CONN_3X2 P201
+L wfred_rev2-rescue:CONN_3X2-conn P201
 U 1 1 5920E592
 P 4400 2150
@@
 SPEED_POWER
 $Comp
-L device:R R204
+L wfred_rev2-rescue:R-device R204
 U 1 1 5BE0AFA5
 P 7450 4900
@@
 	7700 4900 7800 4900
 $Comp
-L atmel:ATMEGA328P-A IC201
+L wfred_rev2-rescue:ATMEGA328P-A-atmel IC201
 U 1 1 5BE1F936
 P 4900 4300
+AR Path="/5BE1F936" Ref="IC201"  Part="1"
+AR Path="/5920C945/5BE1F936" Ref="IC201"  Part="1"
 F 0 "IC201" H 4150 5550 40  0000 L BNN
 F 1 "ATMEGA328P-A" H 5300 2900 40  0000 L BNN

Commit message: Updated schematic to open with kicad 5
Also updated Partlist
Parts:
- D201: symbol my_devices:BAR43 -> wfred_rev2-rescue:BAR43-my_devices
- X201: symbol my_devices:myCRYSTAL -> wfred_rev2-rescue:myCRYSTAL-my_devices
Changed lines of the file:
@@
 F2
 $Comp
-L my_devices:myCRYSTAL X201
+L wfred_rev2-rescue:myCRYSTAL-my_devices X201
 U 1 1 5A171DD9
 P 8400 3500
@@
 	3300 3200 3300 3100
 $Comp
-L my_devices:BAR43 D201
+L wfred_rev2-rescue:BAR43-my_devices D201
 U 1 1 5CD177D6
 P 8100 4600
