File: hardware/wfred-wifi.sch (KiCad schematic (older format))
At the start: 9 parts, among them K401 UART_ESP, K402 UART_AVR, P401 ESP_BOOTLOAD, U401 ESP-12E

Commit message: PCB changes
- Add extra 100uF capacitor for ESP8266 power supply
- Turn battery connector to avoid pushing pins across screw
Parts:
- added C403: 100u, Capacitors_SMD:C_0805_HandSoldering, symbol CAPAPOL
Connections:
- wire segments 29 -> 31
Changed lines of the file:
@@
 $EndComp
 Wire Wire Line
-	1200 2000 1500 2000
+	1200 2000 1800 2000
 Wire Wire Line
 	1500 2000 1500 2200
@@
 	1500 2600 1500 2800
 Wire Wire Line
-	1500 2800 1200 2800
+	1200 2800 1800 2800
 Connection ~ 1200 2800
 NoConn ~ 5200 2500
@@
 NoConn ~ 3400 2400
 NoConn ~ 3400 2300
+$Comp
+L CAPAPOL C403
+U 1 1 5C81829A
+P 1800 2400
+F 0 "C403" H 1850 2500 40  0000 L CNN
+F 1 "100u" H 1850 2300 40  0000 L CNN
+F 2 "Capacitors_SMD:C_0805_HandSoldering" H 1900 2250 30  0000 C CNN
+F 3 "" H 1800 2400 300 0000 C CNN
+	1    1800 2400
+	1    0    0    -1
+$EndComp
+Wire Wire Line
+	1800 2000 1800 2200
+Connection ~ 1500 2000
+Wire Wire Line
+	1800 2800 1800 2600
+Connection ~ 1500 2800
 $EndSCHEMATC

Commit message: Updated schematic and PCB for kicad 5.1.4
Parts:
- C401, C402: symbol C-RESCUE-wfred_rev2 -> wfred_rev2-rescue:C-RESCUE-wfred_rev2
- C403: symbol CAPAPOL -> device:CAPAPOL
- K401, K402: symbol CONN_3 -> conn:CONN_3
- P401: symbol CONN_2 -> conn:CONN_2
- R403, R404, R405: symbol R-RESCUE-wfred_rev2 -> wfred_rev2-rescue:R-RESCUE-wfred_rev2
- U401: symbol ESP-12E -> ESP8266:ESP-12E
Connections:
- wire segments 31 -> 40
Changed lines of the file:
@@
-EESchema Schematic File Version 2
-LIBS:wfred_rev2-rescue
-LIBS:power
-LIBS:device
-LIBS:transistors
-LIBS:conn
-LIBS:linear
-LIBS:regul
-LIBS:74xx
-LIBS:cmos4000
-LIBS:adc-dac
-LIBS:memory
-LIBS:xilinx
-LIBS:microcontrollers
-LIBS:dsp
-LIBS:microchip
-LIBS:analog_switches
-LIBS:motorola
-LIBS:texas
-LIBS:intel
-LIBS:audio
-LIBS:interface
-LIBS:digital-audio
-LIBS:philips
-LIBS:display
-LIBS:cypress
-LIBS:siliconi
-LIBS:opto
-LIBS:atmel
-LIBS:contrib
-LIBS:valves
-LIBS:my_devices
-LIBS:ESP8266
-LIBS:LDL1117S30R
-LIBS:MCP73831T-2ACI_OT
-LIBS:NCV8161BSN300T1G
+EESchema Schematic File Version 4
 LIBS:wfred_rev2-cache
-EELAYER 25 0
+EELAYER 30 0
 EELAYER END
 $Descr A4 11693 8268
@@
 $EndDescr
 $Comp
-L ESP-12E U401
+L ESP8266:ESP-12E U401
 U 1 1 5A11AA62
 P 4300 2600
@@
 NoConn ~ 4550 3500
 $Comp
-L VCC #PWR043
+L power:VCC #PWR043
 U 1 1 5A11E004
 P 2700 1500
@@
 $EndComp
 Wire Wire Line
-	2700 1500 2700 3000
+	2700 1500 2700 2500
 Wire Wire Line
 	2700 3000 3400 3000
@@
 Connection ~ 2700 2500
 $Comp
-L GND-RESCUE-wfred_rev2 #PWR044
+L wfred_rev2-rescue:GND-RESCUE-wfred_rev2 #PWR044
 U 1 1 5A11E30D
 P 6700 3700
@@
 $EndComp
 Wire Wire Line
-	6700 2500 6700 3700
+	6700 2500 6700 2900
 Wire Wire Line
 	6700 3000 5200 3000
 Connection ~ 6700 3000
 $Comp
-L VCC #PWR045
+L power:VCC #PWR045
 U 1 1 5A11E4AA
 P 6300 1550
@@
 	5200 2400 6750 2400
 $Comp
-L CONN_3 K401
+L conn:CONN_3 K401
 U 1 1 5A11EE74
 P 7100 2400
@@
 THIS_TXD
 $Comp
-L CONN_2 P401
+L conn:CONN_2 P401
 U 1 1 5A11F720
 P 7100 2800
@@
 $EndComp
 Wire Wire Line
-	5200 2700 6750 2700
-$Comp
-L GND-RESCUE-wfred_rev2 #PWR046
+	5200 2700 6100 2700
+$Comp
+L wfred_rev2-rescue:GND-RESCUE-wfred_rev2 #PWR046
 U 1 1 5A11FC27
 P 7850 2500
@@
 $EndComp
 $Comp
-L R-RESCUE-wfred_rev2 R403
+L wfred_rev2-rescue:R-RESCUE-wfred_rev2 R403
 U 1 1 5A11FF91
 P 6100 1950
@@
 $EndComp
 $Comp
-L R-RESCUE-wfred_rev2 R404
+L wfred_rev2-rescue:R-RESCUE-wfred_rev2 R404
 U 1 1 5A11FFE4
 P 6100 3350
@@
 $EndComp
 $Comp
-L R-RESCUE-wfred_rev2 R405
+L wfred_rev2-rescue:R-RESCUE-wfred_rev2 R405
 U 1 1 5A120047
 P 6300 1950
@@
 	5200 2900 6100 2900
 $Comp
-L CONN_3 K402
+L conn:CONN_3 K402
 U 1 1 5A11F053
 P 7350 2300
@@
 	6100 1700 6100 1600
 Wire Wire Line
-	6300 1550 6300 1700
+	6300 1550 6300 1600
 Connection ~ 6300 1600
 Wire Wire Line
 	6100 2900 6100 3100
 $Comp
-L GND-RESCUE-wfred_rev2 #PWR047
+L wfred_rev2-rescue:GND-RESCUE-wfred_rev2 #PWR047
 U 1 1 5A120E87
 P 6100 3700
@@
 Connection ~ 6700 2900
 $Comp
-L C-RESCUE-wfred_rev2 C401
+L wfred_rev2-rescue:C-RESCUE-wfred_rev2 C401
 U 1 1 5A127BCA
 P 1200 2400
@@
 $EndComp
 $Comp
-L VCC #PWR048
+L power:VCC #PWR048
 U 1 1 5A127C0E
 P 1200 1800
@@
 $EndComp
 Wire Wire Line
-	1200 1800 1200 2200
-$Comp
-L GND-RESCUE-wfred_rev2 #PWR049
+	1200 1800 1200 2000
+$Comp
+L wfred_rev2-rescue:GND-RESCUE-wfred_rev2 #PWR049
 U 1 1 5A127CDB
 P 1200 2900
@@
 $EndComp
 Wire Wire Line
-	1200 2600 1200 2900
-$Comp
-L C-RESCUE-wfred_rev2 C402
+	1200 2600 1200 2800
+$Comp
+L wfred_rev2-rescue:C-RESCUE-wfred_rev2 C402
 U 1 1 5A199174
 P 1500 2400
@@
 $EndComp
 Wire Wire Line
-	1200 2000 1800 2000
+	1200 2000 1500 2000
 Wire Wire Line
 	1500 2000 1500 2200
@@
 	1500 2600 1500 2800
 Wire Wire Line
-	1200 2800 1800 2800
+	1200 2800 1500 2800
 Connection ~ 1200 2800
 NoConn ~ 5200 2500
@@
 NoConn ~ 3400 2300
 $Comp
-L CAPAPOL C403
+L device:CAPAPOL C403
 U 1 1 5C81829A
 P 1800 2400
@@
 	1800 2800 1800 2600
 Connection ~ 1500 2800
+Wire Wire Line
+	2700 2500 2700 3000
+Wire Wire Line
+	6700 3000 6700 3700
+Wire Wire Line
+	6100 2700 6750 2700
+Wire Wire Line
+	6300 1600 6300 1700
+Wire Wire Line
+	6700 2900 6700 3000
+Wire Wire Line
+	1200 2000 1200 2200
+Wire Wire Line
+	1200 2800 1200 2900
+Wire Wire Line
+	1500 2000 1800 2000
+Wire Wire Line
+	1500 2800 1800 2800
 $EndSCHEMATC

Commit message: Opened schematic and PCB in new kicad version
...causing a couple of changes to libraries and schematic and PCB files
Parts:
- C403: symbol device:CAPAPOL -> wfred_rev2-rescue:CAPAPOL-device
- K401, K402: symbol conn:CONN_3 -> wfred_rev2-rescue:CONN_3-conn
- P401: symbol conn:CONN_2 -> wfred_rev2-rescue:CONN_2-conn
Changed lines of the file:
@@
 EESchema Schematic File Version 4
-LIBS:wfred_rev2-cache
 EELAYER 30 0
 EELAYER END
@@
 	5200 2400 6750 2400
 $Comp
-L conn:CONN_3 K401
+L wfred_rev2-rescue:CONN_3-conn K401
 U 1 1 5A11EE74
 P 7100 2400
@@
 THIS_TXD
 $Comp
-L conn:CONN_2 P401
+L wfred_rev2-rescue:CONN_2-conn P401
 U 1 1 5A11F720
 P 7100 2800
@@
 	5200 2900 6100 2900
 $Comp
-L conn:CONN_3 K402
+L wfred_rev2-rescue:CONN_3-conn K402
 U 1 1 5A11F053
 P 7350 2300
@@
 NoConn ~ 3400 2300
 $Comp
-L device:CAPAPOL C403
+L wfred_rev2-rescue:CAPAPOL-device C403
 U 1 1 5C81829A
 P 1800 2400

Commit message: Updated schematic to open with kicad 5
Also updated Partlist
Parts:
- U401: symbol ESP8266:ESP-12E -> wfred_rev2-rescue:ESP-12E-ESP8266
Changed lines of the file:
@@
 $EndDescr
 $Comp
-L ESP8266:ESP-12E U401
+L wfred_rev2-rescue:ESP-12E-ESP8266 U401
 U 1 1 5A11AA62
 P 4300 2600
