File: hardware/wfred_rev2.sch (KiCad schematic (older format))
At the start: 14 parts, among them CON101 USB-MICRO-B, IC101 MCP73831T-2ACI_OT, IC102 NCV8161BSN300T1G, P101 BATT

Commit message: Opened schematic and PCB in new kicad version
...causing a couple of changes to libraries and schematic and PCB files
Parts:
- C101, C102, C103: symbol device:C -> wfred_rev2-rescue:C-device
- CON101: symbol conn:USB-MINI-B -> wfred_rev2-rescue:USB-MINI-B-conn
- D101, D102: symbol device:LED -> wfred_rev2-rescue:LED-device
- P101: symbol conn:CONN_2 -> wfred_rev2-rescue:CONN_2-conn
- R101, R102, R103, R104: symbol device:R -> wfred_rev2-rescue:R-device
Changed lines of the file:
@@
 EESchema Schematic File Version 4
-LIBS:wfred_rev2-cache
 EELAYER 30 0
 EELAYER END
@@
 $EndSheet
 $Comp
-L conn:CONN_2 P101
+L wfred_rev2-rescue:CONN_2-conn P101
 U 1 1 5BDF535A
 P 1400 1600
@@
 	1750 1500 2800 1500
 $Comp
-L conn:USB-MINI-B CON101
+L wfred_rev2-rescue:USB-MINI-B-conn CON101
 U 1 1 5BDF5403
 P 2050 3500
@@
 $EndComp
 $Comp
-L power:GND #PWR05
+L wfred_rev2-rescue:GND-power #PWR05
 U 1 1 5BDF5538
 P 2800 4200
@@
 Connection ~ 2800 3800
 $Comp
-L power:GND #PWR06
+L wfred_rev2-rescue:GND-power #PWR06
 U 1 1 5BDF55B7
 P 1300 4200
@@
 	4200 1200 4200 2600
 $Comp
-L device:C C101
+L wfred_rev2-rescue:C-device C101
 U 1 1 5BDF64E4
 P 4200 3200
@@
 Connection ~ 4200 2600
 $Comp
-L power:GND #PWR010
+L wfred_rev2-rescue:GND-power #PWR010
 U 1 1 5BDF6575
 P 4200 3600
@@
 	4200 3600 4200 3400
 $Comp
-L power:GND #PWR011
+L wfred_rev2-rescue:GND-power #PWR011
 U 1 1 5BDF65B7
 P 4500 3600
@@
 	4500 2500 4900 2500
 $Comp
-L device:R R101
+L wfred_rev2-rescue:R-device R101
 U 1 1 5BDF69E9
 P 3700 1550
@@
 $EndComp
 $Comp
-L device:R R102
+L wfred_rev2-rescue:R-device R102
 U 1 1 5BDF6A99
 P 3700 3250
@@
 $EndComp
 $Comp
-L device:LED D101
+L wfred_rev2-rescue:LED-device D101
 U 1 1 5BDF6C34
 P 3700 2100
@@
 $EndComp
 $Comp
-L device:LED D102
+L wfred_rev2-rescue:LED-device D102
 U 1 1 5BDF6CF2
 P 3700 2700
@@
 	3700 2900 3700 3000
 $Comp
-L power:GND #PWR012
+L wfred_rev2-rescue:GND-power #PWR012
 U 1 1 5BDF6E99
 P 3700 3600
@@
 	3700 1200 3700 1300
 $Comp
-L device:C C102
+L wfred_rev2-rescue:C-device C102
 U 1 1 5BDF745F
 P 6400 3200
@@
 $EndComp
 $Comp
-L power:GND #PWR014
+L wfred_rev2-rescue:GND-power #PWR014
 U 1 1 5BDF761A
 P 6400 3600
@@
 $EndComp
 $Comp
-L device:R R103
+L wfred_rev2-rescue:R-device R103
 U 1 1 5BDF77A8
 P 6100 3250
@@
 	6100 2500 6100 3000
 $Comp
-L power:GND #PWR016
+L wfred_rev2-rescue:GND-power #PWR016
 U 1 1 5BDF79BD
 P 6100 3600
@@
 	6100 3500 6100 3600
 $Comp
-L device:C C103
+L wfred_rev2-rescue:C-device C103
 U 1 1 5BDF7FBD
 P 7500 2500
@@
 	7500 1200 7500 2300
 $Comp
-L power:GND #PWR018
+L wfred_rev2-rescue:GND-power #PWR018
 U 1 1 5BDF8082
 P 7500 3600
@@
 $EndComp
 $Comp
-L power:GND #PWR022
+L wfred_rev2-rescue:GND-power #PWR022
 U 1 1 5BE0A873
 P 8400 3600
@@
 	9800 2400 9800 3600
 $Comp
-L power:GND #PWR024
+L wfred_rev2-rescue:GND-power #PWR024
 U 1 1 5BE0A9A9
 P 9800 3600
@@
 	8300 2600 8500 2600
 $Comp
-L device:R R104
+L wfred_rev2-rescue:R-device R104
 U 1 1 5CD0A628
 P 10700 2550

Commit message: Updated schematic to open with kicad 5
Also updated Partlist
Parts:
- IC101: symbol MCP73831T-2ACI_OT:MCP73831T-2ACI_OT -> wfred_rev2-rescue:MCP73831T-2ACI_OT-MCP73831T-2ACI_OT
- IC102: symbol NCV8161BSN300T1G:NCV8161BSN300T1G -> wfred_rev2-rescue:NCV8161BSN300T1G-NCV8161BSN300T1G
Changed lines of the file:
@@
 Connection ~ 10400 1400
 $Comp
-L MCP73831T-2ACI_OT:MCP73831T-2ACI_OT IC101
+L wfred_rev2-rescue:MCP73831T-2ACI_OT-MCP73831T-2ACI_OT IC101
 U 1 1 5BDF6387
 P 4900 2400
@@
 $EndComp
 $Comp
-L NCV8161BSN300T1G:NCV8161BSN300T1G IC102
+L wfred_rev2-rescue:NCV8161BSN300T1G-NCV8161BSN300T1G IC102
 U 1 1 5BE0A471
 P 8500 2400
