File: hardware/wfred_rev6.sch (KiCad schematic (older format))
At the start: 18 parts, among them CON101 USB-MICRO-B, IC101 TP4054, IC102 XC6220B331MR, P101 BATT

Commit message: Replace Micro-USB-B with USB-C connector
...including 5k1 resistors for CC-pins
Parts:
- removed CON101: USB-MICRO-B, myFootprints:USB_Micro-B_Molex-105017-0001_longPads, symbol wfred_rev6-rescue:USB-MINI-B-conn-wfred_rev2-rescue
- added J101: USB_C_Receptacle_USB2.0, Connector_USB:USB_C_Receptacle_HRO_TYPE-C-31-M-12, symbol Connector:USB_C_Receptacle_USB2.0
- added R106, R107: 5k1, Resistor_SMD:R_0805_2012Metric_Pad1.15x1.40mm_HandSolder, symbol wfred_rev6-rescue:R-device-wfred_rev2-rescue
Connections:
- wire segments 70 -> 76
- no-connect marks 2 -> 3
Other:
- moved on the sheet: C105, C106, R101, R102

Commit message: Connect USB-C-connector and cleanup
- Replace 2pin + 3pin for RS232 + BOOT with 2x3pin
- Connect USB-C-connector
- Add CC1 and CC2 resistors
- Correct ESP32-S2-WROOM package for hand soldering
- Increase pad sizes for user installed switches / poti
- Correct direction switch pad distance (DRC violation)
- Rearrange some traces and vias
- Add LCSC numbers for pin headers
Parts:
- P101: LCSC (none) -> C706865
Changed lines of the file:
@@
 F 3 "" H 950 1550 60  0001 C CNN
 F 4 "SL 1X36W 2,54" V 950 1550 50  0001 C CNN "Reichelt"
+F 5 "C706865" V 950 1550 50  0001 C CNN "LCSC"
 	1    950  1550
 	-1   0    0    1

Commit message: Update BAT54C order number...
...to one in stock at LCSC
Parts:
- D103: LCSC C375703 -> C556168
Changed lines of the file:
@@
 F 2 "Package_TO_SOT_SMD:SOT-23" H 3475 2825 50  0001 L CNN
 F 3 "http://www.diodes.com/_files/datasheets/ds11005.pdf" H 3320 2700 50  0001 C CNN
-F 4 "C375703" H 3400 2700 50  0001 C CNN "LCSC"
+F 4 "C556168" H 3400 2700 50  0001 C CNN "LCSC"
 F 5 "BAT 54C NXP" H 3400 2700 50  0001 C CNN "Reichelt"
 F 6 "583-BAT54C" H 3400 2700 50  0001 C CNN "Mouser"
