File: hardware/wfred_rev6.sch (KiCad schematic (older format))
At the start: 20 parts, among them IC101 TP4054, IC102 XC6220B331MR, J101 USB_C_Receptacle_USB2.0, P101 BATT

Commit message: Replace out-of-stock components with others
Parts:
- J101: LCSC C393939 -> C165948
- P101: LCSC C706865 -> C492410
Changed lines of the file:
@@
 F 3 "" H 950 1550 60  0001 C CNN
 F 4 "SL 1X36W 2,54" V 950 1550 50  0001 C CNN "Reichelt"
-F 5 "C706865" V 950 1550 50  0001 C CNN "LCSC"
+F 5 "C492410" V 950 1550 50  0001 C CNN "LCSC"
 	1    950  1550
 	-1   0    0    1
@@
 F 2 "Connector_USB:USB_C_Receptacle_HRO_TYPE-C-31-M-12" H 1500 5250 50  0001 C CNN
 F 3 "https://www.usb.org/sites/default/files/documents/usb_type-c.zip" H 1500 5250 50  0001 C CNN
-F 4 "C393939" H 1350 5250 50  0001 C CNN "LCSC"
+F 4 "C165948" H 1350 5250 50  0001 C CNN "LCSC"
 	1    1350 5250
 	1    0    0    -1

Commit message: Change LCSC order number for 22uF caps...
...due to availability.

Also update date and revision number.
Parts:
- C103: LCSC C45783 -> C129303
Changed lines of the file:
@@
 Sheet 1 3
 Title "Wireless FREDI"
-Date "2021-06-28"
-Rev "0.62"
+Date "2022-10-09"
+Rev "0.64"
 Comp "Heiko Rosemann (heiko.rosemann@web.de) CC-BY-SA"
 Comment1 ""
@@
 F 3 "" H 7500 2500 60  0000 C CNN
 F 4 "KEM X5R0805 22U" H 7500 2500 60  0001 C CNN "Reichelt"
-F 5 "C45783" H 7500 2500 50  0001 C CNN "LCSC"
+F 5 "C129303" H 7500 2500 50  0001 C CNN "LCSC"
 F 6 "187-CL21A226MAYNNNE" H 7500 2500 50  0001 C CNN "Mouser"
 F 7 "Mouser 25V, LCSC/Reichelt 6V3" H 7500 2500 50  0001 C CNN "Remark"
