File: hardware/wfred-wifi_rev6.sch (KiCad schematic (older format))
At the start: 14 parts, among them J301 Conn_02x03_Odd_Even, U301 ESP32-S2-WROOM

Commit message: Change LCSC order number for 22uF caps...
...due to availability.

Also update date and revision number.
Parts:
- C304, C305, C306, C307, C308: LCSC C45783 -> C129303
Changed lines of the file:
@@
 Sheet 3 3
 Title "Wireless FREDI"
-Date "2021-06-28"
-Rev "0.62"
+Date "2022-10-09"
+Rev "0.64"
 Comp "Heiko Rosemann (heiko.rosemann@web.de) CC-BY-SA"
 Comment1 ""
@@
 F 3 "" H 7600 4550 60  0000 C CNN
 F 4 "KEM X5R0805 22U" H 7600 4550 60  0001 C CNN "Reichelt"
-F 5 "C45783" H 7600 4550 50  0001 C CNN "LCSC"
+F 5 "C129303" H 7600 4550 50  0001 C CNN "LCSC"
 	1    7600 4550
 	1    0    0    -1
@@
 F 3 "" H 7900 4550 60  0000 C CNN
 F 4 "KEM X5R0805 22U" H 7900 4550 60  0001 C CNN "Reichelt"
-F 5 "C45783" H 7900 4550 50  0001 C CNN "LCSC"
+F 5 "C129303" H 7900 4550 50  0001 C CNN "LCSC"
 	1    7900 4550
 	1    0    0    -1
@@
 F 3 "" H 8200 4550 60  0000 C CNN
 F 4 "KEM X5R0805 22U" H 8200 4550 60  0001 C CNN "Reichelt"
-F 5 "C45783" H 8200 4550 50  0001 C CNN "LCSC"
+F 5 "C129303" H 8200 4550 50  0001 C CNN "LCSC"
 	1    8200 4550
 	1    0    0    -1
@@
 F 3 "" H 8500 4550 60  0000 C CNN
 F 4 "KEM X5R0805 22U" H 8500 4550 60  0001 C CNN "Reichelt"
-F 5 "C45783" H 8500 4550 50  0001 C CNN "LCSC"
+F 5 "C129303" H 8500 4550 50  0001 C CNN "LCSC"
 	1    8500 4550
 	1    0    0    -1
@@
 F 3 "" H 8800 4550 60  0000 C CNN
 F 4 "KEM X5R0805 22U" H 8800 4550 60  0001 C CNN "Reichelt"
-F 5 "C45783" H 8800 4550 50  0001 C CNN "LCSC"
+F 5 "C129303" H 8800 4550 50  0001 C CNN "LCSC"
 	1    8800 4550
 	1    0    0    -1
